File: DesignFiles/_saved_BioVill_Badge.sch (KiCad schematic (older format))
At the start: 136 parts, among them P1 CONN_01X01, P10 CONN_01X01, P11 CONN_01X01, P12 CONN_01X01, P13 ScrewPad1, P14 ScrewPad2, P15 ScrewPad3, P16 ScrewPad4, P2 CONN_01X01, P3 CONN_01X01, P5 CONN_01X01, P6 CONN_01X30, P7 CONN_01X01, P8 CONN_01X01, P9 CONN_01X01, Q1 BSS138, Q2 BSS138, Q3 BSS138, SW1 SW_PUSH, SW2 SW_PUSH, U2 HV507, U3 ARDUINO_MICRO, U6 MCP6002

Commit message: updated parts and added bom draft
Parts:
- C1, C2: renamed from C?; value EGXF251ELL101MU35S -> LGN2W181MELZ45; footprint (none) -> Solutions:Nichcon_LGN_Series_Capacitor_22x45
- D1: renamed from D?; value D_Bridge_+-AA -> CD-MBL110S; footprint (none) -> Solutions:CD-MBLxxxS
- LED1, LED2, LED3, LED4, LED5, LED8: symbol LED -> LED-RESCUE-BioVill_Badge
- R10, R11, R12, R13, R14, R15, R16, R17, R18, R19, R20, R21, R22, R3, R30, R31, R4, R5, R6, R7, R8, R9: symbol R -> R-RESCUE-BioVill_Badge
- gave numbers to parts that had none: 1
Connections:
- net 3.3V: no longer R14.1
Other:
- moved on the sheet: R10, R14
