File: DesignFiles/BioVill_Badge.sch (KiCad schematic (older format))
At the start: 136 parts, among them P1 CONN_01X01, P10 CONN_01X01, P11 CONN_01X01, P12 CONN_01X01, P13 ScrewPad1, P14 ScrewPad2, P15 ScrewPad3, P16 ScrewPad4, P2 CONN_01X01, P3 CONN_01X01, P5 CONN_01X01, P6 CONN_01X30, P7 CONN_01X01, P8 CONN_01X01, P9 CONN_01X01, Q1 BSS138, Q2 BSS138, Q3 BSS138, SW1 SW_PUSH, SW2 SW_PUSH, U2 HV507, U3 ARDUINO_MICRO, U6 MCP6002

Commit message: updated parts and added bom draft
Parts:
- C1, C2: renamed from C?; value EGXF251ELL101MU35S -> LGN2W181MELZ45
- D1: renamed from D?; value D_Bridge_+-AA -> CD-MBL110S; footprint (none) -> Solutions:CD-MBLxxxS
- LED1, LED2, LED3, LED4, LED5, LED8: symbol LED -> LED-RESCUE-BioVill_Badge
- R10, R11, R12, R13, R14, R15, R16, R17, R18, R19, R20, R21, R22, R3, R30, R31, R4, R5, R6, R7, R8, R9: symbol R -> R-RESCUE-BioVill_Badge
- gave numbers to parts that had none: 1

Commit message: minor changes
Parts:
- C1, C2: footprint (none) -> Solutions:Nichcon_LGN_Series_Capacitor_22x45
Connections:
- net 3.3V: no longer R14.1
Other:
- moved on the sheet: R10, R14
Changed lines of the file:
@@
 L R-RESCUE-BioVill_Badge R10
 U 1 1 565C8DD4
-P 11700 5050
-F 0 "R10" V 11600 5050 50  0000 C CNN
-F 1 "10k" V 11700 5050 50  0000 C CNN
-F 2 "Resistors_SMD:R_0805" V 11630 5050 30  0001 C CNN
-F 3 "" H 11700 5050 30  0000 C CNN
-	1    11700 5050
+P 11700 5000
+F 0 "R10" V 11600 5000 50  0000 C CNN
+F 1 "10k" V 11700 5000 50  0000 C CNN
+F 2 "Resistors_SMD:R_0805" V 11630 5000 30  0001 C CNN
+F 3 "" H 11700 5000 30  0000 C CNN
+	1    11700 5000
 	1    0    0    -1
 $EndComp
@@
 L R-RESCUE-BioVill_Badge R14
 U 1 1 565C8A05
-P 12200 4950
-F 0 "R14" V 12100 4950 50  0000 C CNN
-F 1 "10k" V 12200 4950 50  0000 C CNN
-F 2 "Resistors_SMD:R_0805" V 12130 4950 30  0001 C CNN
-F 3 "" H 12200 4950 30  0000 C CNN
-	1    12200 4950
+P 12200 5000
+F 0 "R14" V 12100 5000 50  0000 C CNN
+F 1 "10k" V 12200 5000 50  0000 C CNN
+F 2 "Resistors_SMD:R_0805" V 12130 5000 30  0001 C CNN
+F 3 "" H 12200 5000 30  0000 C CNN
+	1    12200 5000
 	1    0    0    -1
 $EndComp
@@
 	12150 6250 13450 6250
 Wire Wire Line
-	11700 4900 11700 4800
+	11700 4850 11700 4800
 Wire Wire Line
 	10800 5250 11300 5250
@@
 	11950 5200 11950 5150
 Wire Wire Line
-	11700 5250 11700 5200
+	11700 5250 11700 5150
 Wire Wire Line
 	11500 5200 11500 5150
@@
 	11950 4800 11950 4850
 Wire Wire Line
-	11600 4800 12200 4800
+	11600 4800 11950 4800
 Connection ~ 11700 4800
 Wire Wire Line
@@
 	11700 5300 11700 5400
 Wire Wire Line
-	12200 5100 12200 5300
+	12200 5150 12200 5300
 Connection ~ 12200 5300
 Connection ~ 11950 4800
@@
 	11350 1000 11350 1150
 Wire Wire Line
-	11350 1900 11350 1750
+	11350 1750 11350 1900
 $Comp
 L SPST SW3
@@
 F 0 "C1" H 12675 1550 50  0000 L CNN
 F 1 "LGN2W181MELZ45" H 12675 1350 50  0000 L CNN
-F 2 "" H 12650 1450 50  0001 C CNN
-F 3 "" H 12650 1450 50  0001 C CNN
+F 2 "Solutions:Nichcon_LGN_Series_Capacitor_22x45" H 12650 1450 50  0001 C CNN
+F 3 "https://www.mouser.com/ds/2/293/e-lgn-880025.pdf" H 12650 1450 50  0001 C CNN
 	1    12650 1450
 	1    0    0    -1
@@
 F 0 "C2" H 12675 2250 50  0000 L CNN
 F 1 "LGN2W181MELZ45" H 12675 2050 50  0000 L CNN
-F 2 "" H 12650 2150 50  0001 C CNN
+F 2 "Solutions:Nichcon_LGN_Series_Capacitor_22x45" H 12650 2150 50  0001 C CNN
 F 3 "" H 12650 2150 50  0001 C CNN
 	1    12650 2150
