File: DesignFiles/BHV_Badge.sch (KiCad schematic (older format))
At the start: 259 parts, among them J1 USB_C_Receptacle, J2 Conn_02x05_Odd_Even, P1 CONN_01X01, P10 CONN_01X01, P11 CONN_01X01, P12 CONN_01X01, P13 ScrewPad1, P14 ScrewPad2, P15 ScrewPad3, P16 ScrewPad4, P2 ScrewPad4, P3 CONN_01X01, P4 CONN_PSEUDO_AC, P7 CONN_01X01, P8 CONN_01X01, P9 CONN_01X01, SW1 SW_PUSH, SW2 SW_PUSH, SW3 PTS810_SJK_250_SMTR_LFS, SW5 DPDT, T1 TK560P60Y, U1 MAX1771ESA, U10 AQY210EH, U11 AQY210EH, U12 AQY210EH, U13 AQY210EH, U14 TLV1117-33, U15 MCP41010, U16 74xx14, U2 HV507, U3 PAM8301, U4 HV507, U5 SAMD21G18B-A changed from SAM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, U6 MCP6002, U7 HCPL0534, U8 HCPL0534, U9 HCPL0534, Y1 32.765

Commit message: updated USB connector
Parts:
- J1: footprint Connectors_USB:USB_C_Receptacle_Amphenol_12401610E4-2A -> Solutions:USB_C_Receptacle_Amphenol_12401610E4-2A
Changed lines of the file:
@@
 F 0 "J1" H 19850 14200 50  0000 L CNN
 F 1 "USB_C_Receptacle" H 20650 14200 50  0000 R CNN
-F 2 "Connectors_USB:USB_C_Receptacle_Amphenol_12401610E4-2A" H 20400 12750 50  0001 C CNN
+F 2 "Solutions:USB_C_Receptacle_Amphenol_12401610E4-2A" H 20400 12750 50  0001 C CNN
 F 3 "" H 20400 12750 50  0001 C CNN
 	1    20250 12750
@@
 	9450 1350 9450 1700
 $Comp
-L power:GND #PWR?
+L power:GND #PWR0101
 U 1 1 5CEE12F5
 P 10050 2150
-F 0 "#PWR?" H 10050 1900 50  0001 C CNN
+F 0 "#PWR0101" H 10050 1900 50  0001 C CNN
 F 1 "GND" H 10050 2000 50  0000 C CNN
 F 2 "" H 10050 2150 60  0000 C CNN
